File: QuarkCncStepperDrivers.kicad_pcb (KiCad board)
At the start: 4 copper layers, 35.6 x 41.9 mm, 61 parts, among them J1 Conn_01x14, J2 Conn_01x14, Q1 AO4264E, Q2 AO4264E, Q3 AO4264E, Q4 AO4264E, Q5 AO4264E, Q6 AO4264E, Q7 AO4264E, Q8 AO4264E, U1 TMC2160A-TA-T

Commit message: triple connector
Parts:
- removed the R15 at (127.1, 116.3)
- removed the R16 at (130.6, 115.5)
- removed the R17 at (130.7, 116.5)
- removed the R18 at (114.6, 107.7)
- added J2: Conn_01x08, Connector_PinSocket_2.54mm:PinSocket_1x08_P2.54mm_Vertical, F.Cu at (134.6, 104.8)
- J1: value Conn_01x14 -> Conn_02x03_Odd_Even; footprint Connector_PinHeader_2.54mm:PinHeader_1x14_P2.54mm_Vertical -> Connector_PinSocket_2.54mm:PinSocket_2x03_P2.54mm_Vertical
- moved J1 23.0 mm to (111.8, 107.3)
- moved R8 7.27 mm to (117.8, 107.0)
- moved R9 4.95 mm to (114.6, 107.5), turned to 0 degrees
- moved R10 2.57 mm to (111.8, 110.3)
- moved R11 2.05 mm to (108.8, 109.8)
- moved H1 1.03 mm to (103.1, 110.8)
- moved C10 0.93 mm to (107.1, 114.0), turned to -90 degrees
- renumbered J2 to J3, R11 to R10, R12 to R11, R13 to R12, R14 to R13, R19 to R14, R20 to R15, R21 to R16, R22 to R17, R23 to R18, R24 to R19, R25 to R20, R9 to R8, R10 to R9
Connections:
- C12 pad 1: /STEPPER DRIVER X/TMC5160_12VOUT -> +12V
- J1 pad 1: /STEPPER_SCK -> +3V3
- J1 pad 2: /STEPPER_MOSI -> +12V
- J1 pad 3: /STEPPER_MISO -> GND
- J1 pad 4: /STEPPER_X_CSn -> GND
- J1 pad 5: /STEPPER_X_STEP -> VCC
- J1 pad 6: /STEPPER_X_DIR -> VCC
- U1 pad 3: /STEPPER DRIVER X/TMC5160_12VOUT -> +12V
Routing:
- net +3V3: track 26.4 -> 13.6 mm, vias 1 -> 0
- net /STEPPER DRIVER X/TMC5160_12VOUT: track 7.37 -> 0.00 mm
- net /STEPPER_X_CSn: track 12.4 -> 19.5 mm, vias 2 -> 3
- net /STEPPER DRIVER X/VSA: track 9.60 -> 3.12 mm
- net /STEPPER_DIAG2: track 70.9 -> 67.1 mm, vias 2 -> 1
- net /STEPPER_X_ENn: track 20.6 -> 17.6 mm, vias 2 -> 0
- net /STEPPER_X_STEP: track 9.55 -> 6.92 mm
- net +12V: track 25.8 -> 28.2 mm, vias 2 -> 1
- net /STEPPER_X_DIR: track 9.12 -> 6.78 mm
- net /STEPPER DRIVER X/5VOUT: track 27.5 -> 25.8 mm
- net /STEPPER_DIAG1: track 68.5 -> 67.2 mm
- net GND: track 35.7 -> 34.9 mm, vias 32 -> 31
- net VCC: track 4.46 -> 4.00 mm, vias 14 -> 13
Other:
- outline, holes or cut-outs redrawn
