File: stepper_driver.kicad_sch (KiCad schematic)
At the start: 25 parts, among them U1 TMC2160A-TA-T

Commit message: triple connector
Parts:
- removed R15: 0R, Resistor_SMD:R_0402_1005Metric, symbol Device:R
- removed R16, R17: 0R DNI, Resistor_SMD:R_0402_1005Metric, symbol Device:R
- removed R18: 0R DNI, Resistor_SMD:R_0805_2012Metric, symbol Device:R
- renumbered R11 to R10, R12 to R11, R13 to R12, R14 to R13, R9 to R8, R10 to R9
Connections:
- net TMC5160_12VOUT is gone; now on net 12V: C12.1, U1.3 (12VOUT)
Other:
- note removed: "Allow the option to power from 5V for standalone use"
- note removed: "To power from external 12V, install R11, but not R12 and R13"
